File: DesignFiles/ECAD/GateControl/CurrentSense.kicad_sch (KiCad schematic)
At the start: 3 parts, among them U2 INA219AxD

Commit message: finished PCB
Parts:
- renumbered C4_01uF1 to C_IC3
Changed lines of the file:
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@@
   (symbol (lib_id "power:GND") (at 177.8 86.36 0) (unit 1)
     (in_bom yes) (on_board yes) (dnp no) (fields_autoplaced)
-    (property "Reference" "#PWR025" (at 177.8 92.71 0)
+    (property "Reference" "#PWR035" (at 177.8 92.71 0)
       (effects (font (size 1.27 1.27)) hide)
     )
@@
     (instances
       (project "GateControl"
-        (path "/26f853d6-e6b1-4331-a3c6-efb3fa07d05e"
-          (reference "#PWR025") (unit 1)
-        )
-        (path "/26f853d6-e6b1-4331-a3c6-efb3fa07d05e/be56862b-4341-4ca2-aaa8-80cb2fe675d5"
-          (reference "#PWR021") (unit 1)
-        )
         (path "/26f853d6-e6b1-4331-a3c6-efb3fa07d05e/f270a6f3-1404-4f7c-8863-1ec2952f3ed2"
           (reference "#PWR035") (unit 1)
@@
   (symbol (lib_id "power:+3.3V") (at 119.38 68.58 0) (unit 1)
     (in_bom yes) (on_board yes) (dnp no) (fields_autoplaced)
-    (property "Reference" "#PWR019" (at 119.38 72.39 0)
+    (property "Reference" "#PWR031" (at 119.38 72.39 0)
       (effects (font (size 1.27 1.27)) hide)
     )
@@
     (instances
       (project "GateControl"
-        (path "/26f853d6-e6b1-4331-a3c6-efb3fa07d05e"
-          (reference "#PWR019") (unit 1)
-        )
         (path "/26f853d6-e6b1-4331-a3c6-efb3fa07d05e/f270a6f3-1404-4f7c-8863-1ec2952f3ed2"
           (reference "#PWR031") (unit 1)
@@
   (symbol (lib_id "power:+3.3V") (at 177.8 77.47 0) (unit 1)
     (in_bom yes) (on_board yes) (dnp no) (fields_autoplaced)
-    (property "Reference" "#PWR019" (at 177.8 81.28 0)
+    (property "Reference" "#PWR036" (at 177.8 81.28 0)
       (effects (font (size 1.27 1.27)) hide)
     )
@@
     (instances
       (project "GateControl"
-        (path "/26f853d6-e6b1-4331-a3c6-efb3fa07d05e"
-          (reference "#PWR019") (unit 1)
-        )
         (path "/26f853d6-e6b1-4331-a3c6-efb3fa07d05e/f270a6f3-1404-4f7c-8863-1ec2952f3ed2"
           (reference "#PWR036") (unit 1)
@@
   (symbol (lib_id "power:VDC") (at 60.96 71.12 0) (unit 1)
     (in_bom yes) (on_board yes) (dnp no) (fields_autoplaced)
-    (property "Reference" "#PWR02" (at 60.96 73.66 0)
+    (property "Reference" "#PWR07" (at 60.96 73.66 0)
       (effects (font (size 1.27 1.27)) hide)
     )
@@
     (instances
       (project "GateControl"
-        (path "/26f853d6-e6b1-4331-a3c6-efb3fa07d05e/c2c7e3a0-f057-409b-9aed-6370f4d662e9"
-          (reference "#PWR02") (unit 1)
-        )
         (path "/26f853d6-e6b1-4331-a3c6-efb3fa07d05e/f270a6f3-1404-4f7c-8863-1ec2952f3ed2"
           (reference "#PWR07") (unit 1)
@@
   (symbol (lib_id "PCM_Capacitor_AKL:C_Disc_D5.0mm_W2.5mm_P5.00mm") (at 177.8 81.28 0) (unit 1)
     (in_bom yes) (on_board yes) (dnp no)
-    (property "Reference" "C4_01uF1" (at 181.61 80.01 0)
+    (property "Reference" "C_IC3" (at 181.61 80.01 0)
       (effects (font (size 1.27 1.27)) (justify left))
     )
@@
     (instances
       (project "GateControl"
-        (path "/26f853d6-e6b1-4331-a3c6-efb3fa07d05e"
-          (reference "C4_01uF1") (unit 1)
-        )
-        (path "/26f853d6-e6b1-4331-a3c6-efb3fa07d05e/be56862b-4341-4ca2-aaa8-80cb2fe675d5"
-          (reference "C4_01uF1") (unit 1)
-        )
         (path "/26f853d6-e6b1-4331-a3c6-efb3fa07d05e/f270a6f3-1404-4f7c-8863-1ec2952f3ed2"
           (reference "C_IC3") (unit 1)
