File: DesignFiles/ECAD/GateControl/GateControl.kicad_pcb (KiCad board)
At the start: 2 copper layers, 72 x 66.2 mm, 39 parts, among them J3 Conn_01x20_Socket, J5 Conn_01x03_Pin, J6 Conn_01x20_Socket, U1 Pico, U2 INA219AxD, U4 NCP1117-ADJ_SOT223, U5 A4950ELJTR-T-MS

Commit message: finished PCB
Parts:
- removed J3, J6: Conn_01x20_Socket, Connector_PinSocket_2.54mm:PinSocket_1x20_P2.54mm_Vertical
- added C4_01uF1: C_Disc_D5.0mm_W2.5mm_P5.00mm, Capacitor_THT:C_Disc_D5.0mm_W2.5mm_P5.00mm, F.Cu at (196.0, 68.8)
- added D1: LED, LED_SMD:LED_0603_1608Metric_Pad1.05x0.95mm_HandSolder, F.Cu at (204.8, 68.2)
- added D2: 1N4148, Diode_THT:D_DO-35_SOD27_P7.62mm_Horizontal, F.Cu at (175.3, 75.0)
- added D3: 1N4148, Diode_THT:D_DO-35_SOD27_P7.62mm_Horizontal, F.Cu at (158.0, 80.1)
- added D4: 1N4148, Diode_THT:D_DO-35_SOD27_P7.62mm_Horizontal, F.Cu at (167.7, 72.5)
- added D5: 1N4148, Diode_THT:D_DO-35_SOD27_P7.62mm_Horizontal, F.Cu at (155.5, 72.4)
- added IC1: 2521020222501, Samacsys:SON65P200X200X55-7N-D, F.Cu at (198.5, 65.8)
- added R1_1k5: 1k, Resistor_THT:R_Axial_DIN0207_L6.3mm_D2.5mm_P7.62mm_Horizontal, F.Cu at (178.2, 72.2)
- added R2_2k2: 2k, Resistor_THT:R_Axial_DIN0207_L6.3mm_D2.5mm_P7.62mm_Horizontal, F.Cu at (201.2, 72.2)
- added S1: TSC015A03518A, Samacsys:TSC015A03518A, F.Cu at (189.0, 66.0)
- R1_1k1, R1_1k2, R1_1k3, R1_1k4, R2_1k1, R2_2k1, R_LED2: footprint Resistor_THT:R_Axial_DIN0309_L9.0mm_D3.2mm_P12.70mm_Horizontal -> Resistor_THT:R_Axial_DIN0207_L6.3mm_D2.5mm_P7.62mm_Horizontal
- moved R_LED2 12.7 mm to (215.8, 87.6), turned to 90 degrees
- moved C_47uF3 5.39 mm to (165.0, 79.2)
- moved U5 5.20 mm to (161.4, 85.0)
- moved R2_2k1 5.04 mm to (174.8, 97.2)
- moved R1_1k2 4.00 mm to (215.8, 90.2)
- moved R1_1k3 4.00 mm to (211.8, 90.2)
- moved R_SENSE1 3.16 mm to (163.5, 72.0), turned to 45 degrees
- moved H4 1.00 mm to (157.8, 66.0)
- moved H1 0.50 mm to (178.0, 66.0)
- moved H2 0.35 mm to (211.0, 66.0)
- moved C_IC2 0.25 mm to (174.8, 113.0)
Connections:
- J_I2C1 pad 2: +3V3 -> +3.3V
- J_SPI1 pad 2: +3V3 -> +3.3V
- R1_1k2 pad 1: +3V3 -> +3.3V
- R1_1k3 pad 1: +3V3 -> +3.3V
- R1_1k4 pad 1: +3V3 -> +3.3V
- U1 pad 14: Net-(J3-Pin_7) -> unconnected-(U1-GPIO10-Pad14)
- U1 pad 15: Net-(J3-Pin_6) -> unconnected-(U1-GPIO11-Pad15)
- U1 pad 16: Net-(J3-Pin_5) -> unconnected-(U1-GPIO12-Pad16)
- U1 pad 17: Net-(J3-Pin_4) -> unconnected-(U1-GPIO13-Pad17)
- U1 pad 29: Net-(J6-Pin_12) -> unconnected-(U1-GPIO22-Pad29)
- U1 pad 30: Net-(J6-Pin_11) -> unconnected-(U1-RUN-Pad30)
- U1 pad 31: Net-(J6-Pin_10) -> unconnected-(U1-GPIO26_ADC0-Pad31)
- U1 pad 32: Net-(J6-Pin_9) -> unconnected-(U1-GPIO27_ADC1-Pad32)
- U1 pad 34: Net-(J6-Pin_7) -> unconnected-(U1-GPIO28_ADC2-Pad34)
- U1 pad 35: Net-(J6-Pin_6) -> unconnected-(U1-ADC_VREF-Pad35)
- U1 pad 37: Net-(J6-Pin_4) -> unconnected-(U1-3V3_EN-Pad37)
- U1 pad 40: Net-(J6-Pin_1) -> unconnected-(U1-VBUS-Pad40)
Routing:
- net +3.3V: track 0.00 -> 217.5 mm, vias 0 -> 2
- net VDC: track 0.00 -> 66.2 mm
- net /I2C1 SCL: track 0.00 -> 45.3 mm, vias 0 -> 1
- net /IO3: track 0.00 -> 44.2 mm, vias 0 -> 1
- net /I2C1 SDA: track 0.00 -> 43.5 mm, vias 0 -> 2
- net +5V: track 0.00 -> 41.3 mm
- net /Current Sense/DCMotor: track 0.00 -> 31.3 mm
- net /IO2: track 0.00 -> 30.9 mm, vias 0 -> 1
- net GND: track 0.00 -> 30.7 mm, vias 0 -> 17
- net /PWM2: track 0.00 -> 29.9 mm, vias 0 -> 2
- net Net-(S1-COM_1): track 0.00 -> 29.3 mm
- net /PWM1: track 0.00 -> 29.1 mm, vias 0 -> 2
- net Net-(U1-GPIO21): track 0.00 -> 27.9 mm
- net +12V: track 0.00 -> 27.9 mm
- net /I2C0 SDA: track 0.00 -> 26.7 mm
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- added copper zone on F.Cu, net +5V
- added copper zone on B.Cu, net GND
- added copper zone on F.Cu, net GND
Other:
- board size 72 x 66.2 mm -> 72 x 66 mm

Commit message: bla
Parts:
- added 12V1: TestPoint, TestPoint:TestPoint_THTPad_1.0x1.0mm_Drill0.5mm, F.Cu at (158.0, 106.5)
- added 5V1: TestPoint, TestPoint:TestPoint_THTPad_1.0x1.0mm_Drill0.5mm, F.Cu at (177.5, 103.2)
- added D6: LED, LED_SMD:LED_0603_1608Metric_Pad1.05x0.95mm_HandSolder, F.Cu at (174.8, 109.0)
- added D7: LED, LED_SMD:LED_0603_1608Metric_Pad1.05x0.95mm_HandSolder, F.Cu at (172.8, 90.8)
- added G***: LOGO, LOGO, F.Cu at (209.5, 115.2)
- added GND1: TestPoint, TestPoint:TestPoint_THTPad_1.0x1.0mm_Drill0.5mm, F.Cu at (178.2, 113.0)
- added GND2: TestPoint, TestPoint:TestPoint_THTPad_1.0x1.0mm_Drill0.5mm, F.Cu at (166.2, 75.0)
- added GND3: TestPoint, TestPoint:TestPoint_THTPad_1.0x1.0mm_Drill0.5mm, F.Cu at (155.0, 125.0)
- added In1: TestPoint, TestPoint:TestPoint_THTPad_1.0x1.0mm_Drill0.5mm, F.Cu at (179.0, 77.2)
- added In2: TestPoint, TestPoint:TestPoint_THTPad_1.0x1.0mm_Drill0.5mm, F.Cu at (179.0, 79.5)
- added Out1: TestPoint, TestPoint:TestPoint_THTPad_1.0x1.0mm_Drill0.5mm, F.Cu at (174.5, 63.2)
- added Out2: TestPoint, TestPoint:TestPoint_THTPad_1.0x1.0mm_Drill0.5mm, F.Cu at (161.8, 63.5)
- added R10k_4: 2k, Resistor_SMD:R_0805_2012Metric_Pad1.20x1.40mm_HandSolder, F.Cu at (169.0, 91.0)
- added R2k_4: 2k, Resistor_SMD:R_0805_2012Metric_Pad1.20x1.40mm_HandSolder, F.Cu at (175.5, 106.2)
- added Sense1: TestPoint, TestPoint:TestPoint_THTPad_1.0x1.0mm_Drill0.5mm, F.Cu at (162.9, 75.8)
- added VDC1: TestPoint, TestPoint:TestPoint_THTPad_1.0x1.0mm_Drill0.5mm, F.Cu at (155.0, 122.8)
- added VDC2: TestPoint, TestPoint:TestPoint_THTPad_1.0x1.0mm_Drill0.5mm, F.Cu at (174.0, 68.2)
- D2, D3, D4, D5: value 1N4148 -> 1N4001; footprint Diode_THT:D_DO-35_SOD27_P7.62mm_Horizontal -> Diode_THT:D_DO-41_SOD81_P10.16mm_Horizontal
- J_IN1: footprint Connector_BarrelJack:BarrelJack_Kycon_KLDX-0202-xC_Horizontal -> Samacsys:BarrelJack_2,inner_5,5outer_DC-005 2.0
- R2k_1: renamed from R2_2k2; footprint Resistor_THT:R_Axial_DIN0207_L6.3mm_D2.5mm_P7.62mm_Horizontal -> Resistor_SMD:R_0805_2012Metric_Pad1.20x1.40mm_HandSolder
- U4: renamed from U5; footprint Package_SO:SOIC-8-1EP_3.9x4.9mm_P1.27mm_EP2.41x3.3mm -> Samacsys:SOIC8
- moved R1k_2 18.1 mm to (165.4, 93.8), turned to 0 degrees
- moved C_IC1 11.7 mm to (157.8, 103.2)
- moved R1k_3 9.82 mm to (165.4, 96.8), turned to 0 degrees
- moved D2 5.91 mm to (179.7, 71.0)
- moved R1k_1 4.61 mm to (182.8, 71.6), turned to 90 degrees
- moved R2k_1 3.70 mm to (204.8, 71.2)
- moved R2k_3 2.85 mm to (173.0, 99.4)
- moved J_IN1 2.74 mm to (161.6, 122.0)
- moved D4 2.64 mm to (169.7, 74.2)
- moved C_IC4 2.25 mm to (156.0, 89.8)
- moved C_47uF1 2.22 mm to (160.3, 95.5), turned to 0 degrees
- moved U4 2.08 mm to (163.5, 85.0)
- moved D5 2.04 mm to (155.8, 70.4)
- moved C_IC3 1.50 mm to (171.8, 79.2)
- moved C_47uF3 1.35 mm to (166.3, 78.8)
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- renumbered C4_01uF1 to C_IC5, JP4 to JP12, JP6 to JP5, R1_1k2 to R10k_1, R1_1k3 to R10k_2, R1_1k4 to R10k_3, R1_1k5 to R1k_1, R1_1k1 to R1k_2, R2_1k1 to R1k_3, R_LED2 to R2k_2, R2_2k1 to R2k_3, IC1 to U3, U4 to U5
Routing:
- net VDC: track 66.2 -> 7.48 mm
- net +5V: track 41.3 -> 0.01 mm, vias 0 -> 14
- net +12V: track 27.9 -> 12.8 mm
- net GND: track 30.7 -> 17.8 mm, vias 17 -> 32
- net Net-(U5-ADJ): track 20.8 -> 8.31 mm, vias 1 -> 0
- net /Current Sense/DCMotor: track 31.3 -> 39.6 mm
- net /MotorController/Out1: track 24.6 -> 30.9 mm
- net /MotorController/Out2: track 25.1 -> 30.8 mm
- net /PWM1: track 29.1 -> 34.7 mm
- net /PWM2: track 29.9 -> 34.5 mm
- net Net-(D1-A): track 7.39 -> 3.26 mm
- net Net-(U1-GPIO21): track 27.9 -> 30.8 mm, vias 0 -> 2
- net Net-(D7-A): track 0.00 -> 2.08 mm
- net Net-(S1-COM_1): track 29.3 -> 31.3 mm
- net Net-(D6-A): track 0.00 -> 1.93 mm
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- added copper zone on F.Cu, net +12V
- added copper zone on B.Cu, net +5V
- added copper zone on F.Cu, net /Current Sense/DCMotor
- added copper zone on F.Cu, net VDC
Other:
- board text added: "12V"
- board text added: "5V"
- board text added: "G"
