File: DesignFiles/ECAD/GateControl/GateControl.kicad_sch (KiCad schematic)
At the start: 8 parts, among them J3 Conn_01x20_Socket, J5 Conn_01x03_Pin, J6 Conn_01x20_Socket, U1 Pico

Commit message: finished PCB
Parts:
- removed J3, J6: Conn_01x20_Socket, Connector_PinSocket_2.54mm:PinSocket_1x20_P2.54mm_Vertical, symbol Connector:Conn_01x20_Socket
- added C4_01uF1: C_Disc_D5.0mm_W2.5mm_P5.00mm, Capacitor_THT:C_Disc_D5.0mm_W2.5mm_P5.00mm, symbol PCM_Capacitor_AKL:C_Disc_D5.0mm_W2.5mm_P5.00mm
- added D1: LED, LED_SMD:LED_0603_1608Metric_Pad1.05x0.95mm_HandSolder, symbol Device:LED
- added IC1: 2521020222501, Samacsys:SON65P200X200X55-7N-D, symbol Samacsys:2521020222501
- added R1_1k5: 1k, Resistor_THT:R_Axial_DIN0207_L6.3mm_D2.5mm_P7.62mm_Horizontal, symbol Device:R
- added R2_2k2: 2k, Resistor_THT:R_Axial_DIN0207_L6.3mm_D2.5mm_P7.62mm_Horizontal, symbol Device:R
- added S1: TSC015A03518A, Samacsys:TSC015A03518A, symbol Samacsys:TSC015A03518A
Connections:
- net +3.3V: now also C4_01uF1.1, IC1.3 (VDD), R1_1k5.1
- net GND: now also C4_01uF1.2, D1.1 (K), IC1.4 (SAO), IC1.5 (GND), S1.3 (NO_1)
- net I2C1 SCL: now also IC1.1 (SCL)
- net I2C1 SDA: now also IC1.6 (SDA)
- net at U1.26 (GPIO20): now also R1_1k5.2, S1.1 (COM_1)
- net at U1.27 (GPIO21): now also R2_2k2.1
- new net: D1.2 (A), R2_2k2.2
Other:
- note added: "High: device address is 0111000b Low: device address is 0111111b"

Commit message: bla
Parts:
- R2k_1: renamed from R2_2k2; footprint Resistor_THT:R_Axial_DIN0207_L6.3mm_D2.5mm_P7.62mm_Horizontal -> Resistor_SMD:R_0805_2012Metric_Pad1.20x1.40mm_HandSolder
- renumbered C4_01uF1 to C_IC5, R1_1k5 to R1k_1, IC1 to U3
Other:
- moved on the sheet: R1k_1
Changed lines of the file:
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@@
   (junction (at 142.24 128.27) (diameter 0) (color 0 0 0 0)
   )
+  (junction (at 205.74 85.09) (diameter 0) (color 0 0 0 0)
+  )
   (junction (at 115.57 113.03) (diameter 0) (color 0 0 0 0)
   )
@@
   (junction (at 248.92 33.02) (diameter 0) (color 0 0 0 0)
   )
-  (junction (at 212.09 85.09) (diameter 0) (color 0 0 0 0)
-  )
   (wire (pts (xy 166.37 87.63) (xy 166.37 100.33))
     (stroke (width 0) (type default))
@@
     (stroke (width 0) (type default))
   )
+  (wire (pts (xy 205.74 85.09) (xy 187.96 85.09))
+    (stroke (width 0) (type default))
+  )
+  (wire (pts (xy 205.74 85.09) (xy 212.09 85.09))
+    (stroke (width 0) (type default))
+  )
   (wire (pts (xy 160.02 102.87) (xy 209.55 102.87))
     (stroke (width 0) (type default))
@@
   )
   (wire (pts (xy 124.46 87.63) (xy 115.57 87.63))
-    (stroke (width 0) (type default))
-  )
-  (wire (pts (xy 212.09 85.09) (xy 187.96 85.09))
     (stroke (width 0) (type default))
   )
@@
     )
   )
-  (symbol (lib_id "power:+3.3V") (at 212.09 77.47 0) (unit 1)
-    (in_bom yes) (on_board yes) (dnp no) (fields_autoplaced)
-    (property "Reference" "#PWR04" (at 212.09 81.28 0)
-      (effects (font (size 1.27 1.27)) hide)
-    )
-    (property "Value" "+3.3V" (at 212.09 72.39 0)
-      (effects (font (size 1.27 1.27)))
-    )
-    (property "Footprint" "" (at 212.09 77.47 0)
-      (effects (font (size 1.27 1.27)) hide)
-    )
-    (property "Datasheet" "" (at 212.09 77.47 0)
+  (symbol (lib_id "power:+3.3V") (at 205.74 77.47 0) (unit 1)
+    (in_bom yes) (on_board yes) (dnp no) (fields_autoplaced)
+    (property "Reference" "#PWR04" (at 205.74 81.28 0)
+      (effects (font (size 1.27 1.27)) hide)
+    )
+    (property "Value" "+3.3V" (at 205.74 72.39 0)
+      (effects (font (size 1.27 1.27)))
+    )
+    (property "Footprint" "" (at 205.74 77.47 0)
+      (effects (font (size 1.27 1.27)) hide)
+    )
+    (property "Datasheet" "" (at 205.74 77.47 0)
       (effects (font (size 1.27 1.27)) hide)
     )
@@
   (symbol (lib_id "Device:R") (at 213.36 104.14 90) (unit 1)
     (in_bom yes) (on_board yes) (dnp no) (fields_autoplaced)
-    (property "Reference" "R2_2k2" (at 213.36 97.79 90)
+    (property "Reference" "R2k_1" (at 213.36 97.79 90)
       (effects (font (size 1.27 1.27)))
     )
@@
       (effects (font (size 1.27 1.27)))
     )
-    (property "Footprint" "Resistor_THT:R_Axial_DIN0207_L6.3mm_D2.5mm_P7.62mm_Horizontal" (at 213.36 105.918 90)
+    (property "Footprint" "Resistor_SMD:R_0805_2012Metric_Pad1.20x1.40mm_HandSolder" (at 213.36 105.918 90)
       (effects (font (size 1.27 1.27)) hide)
     )
@@
       (project "GateControl"
         (path "/26f853d6-e6b1-4331-a3c6-efb3fa07d05e"
-          (reference "R2_2k2") (unit 1)
+          (reference "R2k_1") (unit 1)
         )
       )
@@
   (symbol (lib_id "PCM_Capacitor_AKL:C_Disc_D5.0mm_W2.5mm_P5.00mm") (at 205.74 39.37 0) (unit 1)
     (in_bom yes) (on_board yes) (dnp no)
-    (property "Reference" "C4_01uF1" (at 209.55 38.1 0)
+    (property "Reference" "C_IC5" (at 209.55 38.1 0)
       (effects (font (size 1.27 1.27)) (justify left))
     )
@@
       (project "GateControl"
         (path "/26f853d6-e6b1-4331-a3c6-efb3fa07d05e"
-          (reference "C4_01uF1") (unit 1)
+          (reference "C_IC5") (unit 1)
         )
       )
@@
   (symbol (lib_id "Samacsys:2521020222501") (at 223.52 27.94 0) (unit 1)
     (in_bom yes) (on_board yes) (dnp no) (fields_autoplaced)
-    (property "Reference" "IC1" (at 236.22 20.32 0)
+    (property "Reference" "U3" (at 236.22 20.32 0)
       (effects (font (size 1.27 1.27)))
     )
@@
       (project "GateControl"
         (path "/26f853d6-e6b1-4331-a3c6-efb3fa07d05e"
-          (reference "IC1") (unit 1)
+          (reference "U3") (unit 1)
         )
       )
@@
     )
   )
-  (symbol (lib_id "Device:R") (at 212.09 81.28 0) (unit 1)
-    (in_bom yes) (on_board yes) (dnp no) (fields_autoplaced)
-    (property "Reference" "R1_1k5" (at 214.63 80.01 0)
+  (symbol (lib_id "Device:R") (at 205.74 81.28 0) (unit 1)
+    (in_bom yes) (on_board yes) (dnp no) (fields_autoplaced)
+    (property "Reference" "R1k_1" (at 208.28 80.01 0)
       (effects (font (size 1.27 1.27)) (justify left))
     )
-    (property "Value" "1k" (at 214.63 82.55 0)
+    (property "Value" "1k" (at 208.28 82.55 0)
       (effects (font (size 1.27 1.27)) (justify left))
     )
-    (property "Footprint" "Resistor_THT:R_Axial_DIN0207_L6.3mm_D2.5mm_P7.62mm_Horizontal" (at 210.312 81.28 90)
-      (effects (font (size 1.27 1.27)) hide)
-    )
-    (property "Datasheet" "~" (at 212.09 81.28 0)
+    (property "Footprint" "Resistor_THT:R_Axial_DIN0207_L6.3mm_D2.5mm_P7.62mm_Horizontal" (at 203.962 81.28 90)
+      (effects (font (size 1.27 1.27)) hide)
+    )
+    (property "Datasheet" "~" (at 205.74 81.28 0)
       (effects (font (size 1.27 1.27)) hide)
     )
@@
       (project "GateControl"
         (path "/26f853d6-e6b1-4331-a3c6-efb3fa07d05e"
-          (reference "R1_1k5") (unit 1)
-        )
-      )
+          (reference "R1k_1") (unit 1)
+        )
+      )
