File: DesignFiles/ECAD/GateControl/LDO.kicad_sch (KiCad schematic)
At the start: 8 parts, among them U4 NCP1117-ADJ_SOT223

Commit message: finished PCB
Parts:
- R1_1k1: renamed from R3_2k1; footprint Resistor_THT:R_Axial_DIN0309_L9.0mm_D3.2mm_P12.70mm_Horizontal -> Resistor_THT:R_Axial_DIN0207_L6.3mm_D2.5mm_P7.62mm_Horizontal
- R2_1k1: renamed from R1_1k1; footprint Resistor_THT:R_Axial_DIN0309_L9.0mm_D3.2mm_P12.70mm_Horizontal -> Resistor_THT:R_Axial_DIN0207_L6.3mm_D2.5mm_P7.62mm_Horizontal
- R2_2k1: footprint Resistor_THT:R_Axial_DIN0309_L9.0mm_D3.2mm_P12.70mm_Horizontal -> Resistor_THT:R_Axial_DIN0207_L6.3mm_D2.5mm_P7.62mm_Horizontal
- renumbered C1_47uF1 to C_47uF1, C1_47uF1 to C_47uF2, C3_01uF1 to C_IC1, C4_01uF1 to C_IC2

Commit message: bla
Parts:
- added 12V1, 5V1, GND1: TestPoint, TestPoint:TestPoint_THTPad_1.0x1.0mm_Drill0.5mm, symbol Connector:TestPoint
- added D6: LED, LED_SMD:LED_0603_1608Metric_Pad1.05x0.95mm_HandSolder, symbol Device:LED
- added R2k_4: 2k, Resistor_SMD:R_0805_2012Metric_Pad1.20x1.40mm_HandSolder, symbol Device:R
- renumbered R1_1k1 to R1k_2, R2_1k1 to R1k_3, R2_2k1 to R2k_3, U4 to U5
Connections:
- net +12V: now also 12V1.1
- net +5V: now also 5V1.1, R2k_4.1
- net GND: now also D6.1 (K), GND1.1
- new net: D6.2 (A), R2k_4.2
