File: DesignFiles/ECAD/GateControl/MotorController.kicad_sch (KiCad schematic)
At the start: 4 parts, among them U5 A4950ELJTR-T-MS

Commit message: finished PCB
Parts:
- added D2, D3, D4, D5: 1N4148, Diode_THT:D_DO-35_SOD27_P7.62mm_Horizontal, symbol Diode:1N4148
- renumbered C1_47uF1 to C_47uF3, C4_01uF1 to C_IC4, R_SHNT to R_SENSE1
Connections:
- net DCMotor: now also D2.1 (K), D3.1 (K)
- net GND: now also D4.2 (A), D5.2 (A)
- net Out1: now also D2.2 (A), D4.1 (K)
- net Out2: now also D3.2 (A), D5.1 (K)
Other:
- moved on the sheet: C_47uF3

Commit message: bla
Parts:
- removed D2, D3, D4, D5: 1N4148, Diode_THT:D_DO-35_SOD27_P7.62mm_Horizontal, symbol Diode:1N4148
- added D2, D3, D4, D5: 1N4001, Diode_THT:D_DO-41_SOD81_P10.16mm_Horizontal, symbol Diode:1N4001
- added GND2, In1, In2, Out1, Out2, Sense1, VDC2: TestPoint, TestPoint:TestPoint_THTPad_1.0x1.0mm_Drill0.5mm, symbol Connector:TestPoint
- U4: renamed from U5; footprint Package_SO:SOIC-8-1EP_3.9x4.9mm_P1.27mm_EP2.41x3.3mm -> Samacsys:SOIC8
Connections:
- net DCMotor: now also D2.1 (K), D3.1 (K), VDC2.1
- net GND: now also D4.2 (A), D5.2 (A), GND2.1
- net In1: now also In1.1
- net In2: now also In2.1
- net Out1: now also D2.2 (A), D4.1 (K), Out1.1
- net Out2: now also D3.2 (A), D5.1 (K), Out2.1
- net at R_SENSE1.1, U4.7 (LSS): now also Sense1.1
Other:
- moved on the sheet: C_IC4
