File: DesignFiles/ECAD/GateControl/Outputs.kicad_sch (KiCad schematic)
At the start: 11 parts

Commit message: finished PCB
Parts:
- R1_1k2, R1_1k3, R1_1k4: renamed from R1_1k1; footprint Resistor_THT:R_Axial_DIN0309_L9.0mm_D3.2mm_P12.70mm_Horizontal -> Resistor_THT:R_Axial_DIN0207_L6.3mm_D2.5mm_P7.62mm_Horizontal
- R_LED2: renamed from R2_2k1; footprint Resistor_THT:R_Axial_DIN0309_L9.0mm_D3.2mm_P12.70mm_Horizontal -> Resistor_THT:R_Axial_DIN0207_L6.3mm_D2.5mm_P7.62mm_Horizontal
- renumbered J_IN2 to J_BTN1, J_IN2 to J_BTN2, J_IN2 to J_BTN3, J_IN2 to J_LED1, J_IN2 to J_Motor1
Connections:
- net +3V3 renamed +3.3V

Commit message: bla
Parts:
- renumbered R1_1k2 to R10k_1, R1_1k3 to R10k_2, R1_1k4 to R10k_3, R_LED2 to R2k_2
Changed lines of the file:
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@@
   (symbol (lib_id "Device:R") (at 77.47 38.1 0) (unit 1)
     (in_bom yes) (on_board yes) (dnp no) (fields_autoplaced)
-    (property "Reference" "R1_1k3" (at 80.01 36.83 0)
+    (property "Reference" "R10k_2" (at 80.01 36.83 0)
       (effects (font (size 1.27 1.27)) (justify left))
     )
@@
       (project "GateControl"
         (path "/26f853d6-e6b1-4331-a3c6-efb3fa07d05e/bd3f696f-e467-435d-89b5-b76fd58161f1"
-          (reference "R1_1k3") (unit 1)
+          (reference "R10k_2") (unit 1)
         )
       )
@@
   (symbol (lib_id "Device:R") (at 40.64 38.1 0) (unit 1)
     (in_bom yes) (on_board yes) (dnp no) (fields_autoplaced)
-    (property "Reference" "R1_1k2" (at 43.18 36.83 0)
+    (property "Reference" "R10k_1" (at 43.18 36.83 0)
       (effects (font (size 1.27 1.27)) (justify left))
     )
@@
       (project "GateControl"
         (path "/26f853d6-e6b1-4331-a3c6-efb3fa07d05e/bd3f696f-e467-435d-89b5-b76fd58161f1"
-          (reference "R1_1k2") (unit 1)
+          (reference "R10k_1") (unit 1)
         )
       )
@@
   (symbol (lib_id "Device:R") (at 121.92 38.1 0) (unit 1)
     (in_bom yes) (on_board yes) (dnp no) (fields_autoplaced)
-    (property "Reference" "R1_1k4" (at 124.46 36.83 0)
+    (property "Reference" "R10k_3" (at 124.46 36.83 0)
       (effects (font (size 1.27 1.27)) (justify left))
     )
@@
       (project "GateControl"
         (path "/26f853d6-e6b1-4331-a3c6-efb3fa07d05e/bd3f696f-e467-435d-89b5-b76fd58161f1"
-          (reference "R1_1k4") (unit 1)
+          (reference "R10k_3") (unit 1)
         )
       )
@@
   (symbol (lib_id "Device:R") (at 34.29 77.47 90) (unit 1)
     (in_bom yes) (on_board yes) (dnp no) (fields_autoplaced)
-    (property "Reference" "R_LED2" (at 34.29 71.12 90)
+    (property "Reference" "R2k_2" (at 34.29 71.12 90)
       (effects (font (size 1.27 1.27)))
     )
@@
       (project "GateControl"
         (path "/26f853d6-e6b1-4331-a3c6-efb3fa07d05e/bd3f696f-e467-435d-89b5-b76fd58161f1"
-          (reference "R_LED2") (unit 1)
-        )
-      )
+          (reference "R2k_2") (unit 1)
+        )
+      )
