File: DesignFiles/ECAD/GateControl/PowerIn.kicad_sch (KiCad schematic)
At the start: 5 parts

Commit message: finished PCB
Parts:
- renumbered D1_TVS1 to D_TVS1, JP2 to JP4, JP4 to JP6

Commit message: bla
Parts:
- added D7: LED, LED_SMD:LED_0603_1608Metric_Pad1.05x0.95mm_HandSolder, symbol Device:LED
- added GND3, VDC1: TestPoint, TestPoint:TestPoint_THTPad_1.0x1.0mm_Drill0.5mm, symbol Connector:TestPoint
- added R10k_4: 2k, Resistor_SMD:R_0805_2012Metric_Pad1.20x1.40mm_HandSolder, symbol Device:R
- J_IN1: footprint Connector_BarrelJack:BarrelJack_Kycon_KLDX-0202-xC_Horizontal -> Samacsys:BarrelJack_2,inner_5,5outer_DC-005 2.0
- renumbered JP4 to JP12, JP6 to JP5
Connections:
- net GND: now also D7.1 (K), GND3.1
- net VDC: now also R10k_4.1, VDC1.1
- new net: D7.2 (A), R10k_4.2
Changed lines of the file:
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@@
 (kicad_sch (version 20230121) (generator eeschema)
   (paper "A4")
+  (junction (at 52.07 48.26) (diameter 0) (color 0 0 0 0)
+  )
   (junction (at 102.87 43.18) (diameter 0) (color 0 0 0 0)
   )
@@
   (junction (at 71.12 43.18) (diameter 0) (color 0 0 0 0)
   )
+  (junction (at 111.76 43.18) (diameter 0) (color 0 0 0 0)
+  )
+  (junction (at 90.17 43.18) (diameter 0) (color 0 0 0 0)
+  )
   (junction (at 77.47 43.18) (diameter 0) (color 0 0 0 0)
   )
@@
     (stroke (width 0) (type default))
   )
-  (wire (pts (xy 77.47 43.18) (xy 102.87 43.18))
+  (wire (pts (xy 77.47 43.18) (xy 90.17 43.18))
     (stroke (width 0) (type default))
   )
@@
     (stroke (width 0) (type default))
   )
+  (wire (pts (xy 111.76 43.18) (xy 114.3 43.18))
+    (stroke (width 0) (type default))
+  )
   (wire (pts (xy 71.12 43.18) (xy 77.47 43.18))
     (stroke (width 0) (type default))
@@
     (stroke (width 0) (type default))
   )
-  (wire (pts (xy 102.87 43.18) (xy 114.3 43.18))
+  (wire (pts (xy 90.17 43.18) (xy 102.87 43.18))
+    (stroke (width 0) (type default))
+  )
+  (wire (pts (xy 102.87 43.18) (xy 111.76 43.18))
     (stroke (width 0) (type default))
   )
@@
     (effects (font (size 1.27 1.27)) (justify left))
   )
+  (symbol (lib_id "Connector:TestPoint") (at 111.76 43.18 0) (unit 1)
+    (in_bom yes) (on_board yes) (dnp no) (fields_autoplaced)
+    (property "Reference" "VDC1" (at 114.3 38.608 0)
+      (effects (font (size 1.27 1.27)) (justify left))
+    )
+    (property "Value" "TestPoint" (at 114.3 41.148 0)
+      (effects (font (size 1.27 1.27)) (justify left))
+    )
+    (property "Footprint" "TestPoint:TestPoint_THTPad_1.0x1.0mm_Drill0.5mm" (at 116.84 43.18 0)
+      (effects (font (size 1.27 1.27)) hide)
+    )
+    (property "Datasheet" "~" (at 116.84 43.18 0)
+      (effects (font (size 1.27 1.27)) hide)
+    )
+    (pin "1")
+    (instances
+      (project "GateControl"
+        (path "/26f853d6-e6b1-4331-a3c6-efb3fa07d05e/c2c7e3a0-f057-409b-9aed-6370f4d662e9"
+          (reference "VDC1") (unit 1)
+        )
+      )
+    )
+  )
   (symbol (lib_id "Connector:Conn_01x02_Pin") (at 119.38 45.72 180) (unit 1)
     (in_bom yes) (on_board yes) (dnp no) (fields_autoplaced)
@@
   (symbol (lib_id "Jumper:SolderJumper_2_Open") (at 77.47 34.29 270) (unit 1)
     (in_bom yes) (on_board yes) (dnp no) (fields_autoplaced)
-    (property "Reference" "JP6" (at 80.01 33.02 90)
+    (property "Reference" "JP5" (at 80.01 33.02 90)
       (effects (font (size 1.27 1.27)) (justify left))
     )
@@
       (project "GateControl"
         (path "/26f853d6-e6b1-4331-a3c6-efb3fa07d05e/c2c7e3a0-f057-409b-9aed-6370f4d662e9"
-          (reference "JP6") (unit 1)
+          (reference "JP5") (unit 1)
         )
       )
@@
     )
   )
+  (symbol (lib_id "Device:R") (at 90.17 46.99 0) (unit 1)
+    (in_bom yes) (on_board yes) (dnp no) (fields_autoplaced)
+    (property "Reference" "R10k_4" (at 92.71 45.72 0)
+      (effects (font (size 1.27 1.27)) (justify left))
+    )
+    (property "Value" "2k" (at 92.71 48.26 0)
+      (effects (font (size 1.27 1.27)) (justify left))
+    )
+    (property "Footprint" "Resistor_SMD:R_0805_2012Metric_Pad1.20x1.40mm_HandSolder" (at 88.392 46.99 90)
+      (effects (font (size 1.27 1.27)) hide)
+    )
+    (property "Datasheet" "~" (at 90.17 46.99 0)
+      (effects (font (size 1.27 1.27)) hide)
+    )
+    (pin "1")
+    (pin "2")
+    (instances
+      (project "GateControl"
+        (path "/26f853d6-e6b1-4331-a3c6-efb3fa07d05e/c2c7e3a0-f057-409b-9aed-6370f4d662e9"
+          (reference "R10k_4") (unit 1)
+        )
+      )
+    )
+  )
   (symbol (lib_id "Connector:Barrel_Jack") (at 40.64 45.72 0) (unit 1)
     (in_bom yes) (on_board yes) (dnp no) (fields_autoplaced)
@@
       (effects (font (size 1.27 1.27)))
     )
-    (property "Footprint" "Connector_BarrelJack:BarrelJack_Kycon_KLDX-0202-xC_Horizontal" (at 41.91 46.736 0)
+    (property "Footprint" "Samacsys:BarrelJack_2,inner_5,5outer_DC-005 2.0" (at 41.91 46.736 0)
       (effects (font (size 1.27 1.27)) hide)
     )
@@
     )
   )
+  (symbol (lib_id "Connector:TestPoint") (at 52.07 48.26 270) (unit 1)
+    (in_bom yes) (on_board yes) (dnp no) (fields_autoplaced)
+    (property "Reference" "GND3" (at 57.15 46.99 90)
+      (effects (font (size 1.27 1.27)) (justify left))
+    )
+    (property "Value" "TestPoint" (at 57.15 49.53 90)
+      (effects (font (size 1.27 1.27)) (justify left))
+    )
+    (property "Footprint" "TestPoint:TestPoint_THTPad_1.0x1.0mm_Drill0.5mm" (at 52.07 53.34 0)
+      (effects (font (size 1.27 1.27)) hide)
+    )
+    (property "Datasheet" "~" (at 52.07 53.34 0)
+      (effects (font (size 1.27 1.27)) hide)
+    )
+    (pin "1")
+    (instances
+      (project "GateControl"
+        (path "/26f853d6-e6b1-4331-a3c6-efb3fa07d05e/c2c7e3a0-f057-409b-9aed-6370f4d662e9"
+          (reference "GND3") (unit 1)
+        )
+      )
+    )
+  )
+  (symbol (lib_id "Device:LED") (at 90.17 54.61 90) (unit 1)
+    (in_bom yes) (on_board yes) (dnp no) (fields_autoplaced)
+    (property "Reference" "D7" (at 93.98 54.9275 90)
+      (effects (font (size 1.27 1.27)) (justify right))
+    )
+    (property "Value" "LED" (at 93.98 57.4675 90)
+      (effects (font (size 1.27 1.27)) (justify right))
+    )
+    (property "Footprint" "LED_SMD:LED_0603_1608Metric_Pad1.05x0.95mm_HandSolder" (at 90.17 54.61 0)
+      (effects (font (size 1.27 1.27)) hide)
+    )
+    (property "Datasheet" "~" (at 90.17 54.61 0)
+      (effects (font (size 1.27 1.27)) hide)
+    )
+    (pin "1")
+    (pin "2")
+    (instances
+      (project "GateControl"
+        (path "/26f853d6-e6b1-4331-a3c6-efb3fa07d05e/c2c7e3a0-f057-409b-9aed-6370f4d662e9"
+          (reference "D7") (unit 1)
+        )
+      )
+    )
+  )
   (symbol (lib_id "Jumper:SolderJumper_2_Open") (at 52.07 34.29 270) (unit 1)
     (in_bom yes) (on_board yes) (dnp no) (fields_autoplaced)
-    (property "Reference" "JP4" (at 54.61 33.02 90)
+    (property "Reference" "JP12" (at 54.61 33.02 90)
       (effects (font (size 1.27 1.27)) (justify left))
     )
@@
       (project "GateControl"
         (path "/26f853d6-e6b1-4331-a3c6-efb3fa07d05e/c2c7e3a0-f057-409b-9aed-6370f4d662e9"
-          (reference "JP4") (unit 1)
+          (reference "JP12") (unit 1)
         )
       )
@@
         )
       )
+    )
+  )
+  (symbol (lib_id "power:GND") (at 90.17 58.42 0) (unit 1)
+    (in_bom yes) (on_board yes) (dnp no) (fields_autoplaced)
+    (property "Reference" "#PWR055" (at 90.17 64.77 0)
+      (effects (font (size 1.27 1.27)) hide)
+    )
+    (property "Value" "GND" (at 90.17 63.5 0)
+      (effects (font (size 1.27 1.27)))
+    )
+    (property "Footprint" "" (at 90.17 58.42 0)
+      (effects (font (size 1.27 1.27)) hide)
+    )
+    (property "Datasheet" "" (at 90.17 58.42 0)
+      (effects (font (size 1.27 1.27)) hide)
+    )
+    (pin "1")
+    (instances
+      (project "GateControl"
+        (path "/26f853d6-e6b1-4331-a3c6-efb3fa07d05e/c2c7e3a0-f057-409b-9aed-6370f4d662e9"
+          (reference "#PWR055") (unit 1)
+        )
+      )
